File: electronics/rove_v/rove_v.kicad_sch (KiCad schematic)
At the start: 28 parts, among them J1 USB-C, J2 Battery, J3 LeftMotor, J4 RightMotor, SW1 BOOT, SW2 RST, U1 ESP32-S3-WROOM-1, U2 XC6220B331MR, U3 DRV8833PW, U4 TP4056

Commit message: Add ROVE-V completed PCB, docs, tools, and Gerbers
- PCB resized 100×80mm → 60×50mm (62% area reduction)
- Fully routed with freerouting, all DRC violations fixed manually
- DRU custom rules: JLCPCB 0.127mm min clearance + J1 USB-C override
- Final DRC: 145 violations (all J1 connector geometry), 0 unconnected
- Gerbers generated and ready for JLCPCB (rove_v_gerbers_drc_clean.zip)
- board_specs.md: ROVE-V section corrected (DW01A+FS8205A, no TP4056)
- tools/: export_dsn.py, import_ses.py, resize_board_60x50.py, etc.

Co-Authored-By: Claude Sonnet 4.6 <noreply@anthropic.com>
Parts:
- removed U4: TP4056, Package_SO:SOP-8_3.9x4.9mm_P1.27mm, symbol Custom:TP4056
- added Q1: FS8205A, Package_TO_SOT_SMD:SOT-23-6, symbol Custom:FS8205A
- added R6: 100k, Resistor_SMD:R_0402_1005Metric, symbol Device:R
- added R7: 47k, Resistor_SMD:R_0402_1005Metric, symbol Device:R
- added U5: DW01A, Package_TO_SOT_SMD:SOT-23-6, symbol Custom:DW01A
Connections:
- net USB_5V: no longer J1.A4 (VBUS), J1.A9 (VBUS), J1.B4 (VBUS), J1.B9 (VBUS)
- new net: J1.A4 (VBUS), J1.A9 (VBUS), J1.B4 (VBUS), J1.B9 (VBUS)
Other:
- note added: "Battery protection: DW01A + FS8205A BATT_RAW: unprotected battery input VBAT: protected output to rest of circuit VBAT_MON → ESP32 GPIO10 (ADC1_CH9) VBAT_MON = VBAT × 47/(100+47) ≈ VBAT × 0.32 Low battery threshold: VBAT_MON < 1.06V → VBAT < 3.3V"
Changed lines of the file:
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@@
 (kicad_sch
 	(version 20231120)
-	(generator "voice_car_generator")
-	(generator_version "1.0")
+	(generator "rove_v_r2")
+	(generator_version "2.0")
 	(uuid "vc001111-2222-3333-4444-555566667777")
 	(paper "A4")
@@
 		)
 	)
-	(label "USB_5V"
-		(at 52.78 99.76 0)
-		(effects
-			(font
-				(size 1.27 1.27)
-			)
-			(justify left bottom)
-		)
-	)
-	(label "USB_5V"
-		(at 52.78 99.76 0)
-		(effects
-			(font
-				(size 1.27 1.27)
-			)
-			(justify left bottom)
-		)
-	)
-	(label "USB_5V"
-		(at 52.78 99.76 0)
-		(effects
-			(font
-				(size 1.27 1.27)
-			)
-			(justify left bottom)
-		)
-	)
-	(label "USB_5V"
-		(at 52.78 99.76 0)
-		(effects
-			(font
-				(size 1.27 1.27)
-			)
-			(justify left bottom)
-		)
-	)
 	(label "USB_D+"
 		(at 52.78 117.54 0)
@@
 	)
 	(symbol
-		(lib_id "Custom:TP4056")
-		(at 55 45 0)
-		(unit 1)
-		(exclude_from_sim no)
-		(in_bom yes)
-		(on_board yes)
-		(dnp no)
-		(property "Reference" "U4"
-			(at 55 37.5 0)
-			(effects (font (size 1.27 1.27)))
-		)
-		(property "Value" "TP4056"
-			(at 55 39.0 0)
-			(effects (font (size 1.27 1.27)))
-		)
-		(property "Footprint" "Package_SO:SOP-8_3.9x4.9mm_P1.27mm"
-			(at 55 45 0)
-			(effects (font (size 1.27 1.27)) (hide yes))
-		)
-		(property "Datasheet" "~"
-			(at 55 45 0)
-			(effects (font (size 1.27 1.27)) (hide yes))
-		)
-		(property "Description" ""
-			(at 55 45 0)
-			(effects (font (size 1.27 1.27)) (hide yes))
-		)
-		(pin "1")
-		(pin "2")
-		(pin "3")
-		(pin "4")
-		(pin "5")
-		(pin "6")
-		(pin "7")
-		(pin "8")
-		(instances
-			(project ""
-				(path "/voice-car-001"
-					(reference "U4")
-					(unit 1)
-				)
-			)
-		)
-	)
-	(symbol
 		(lib_id "Custom:INMP441")
 		(at 155 175 0)
@@
 		)
 	)
+	(symbol
+		(lib_id "Custom:DW01A")
+		(at 55 100 0)
+		(unit 1)
+		(exclude_from_sim no)
+		(in_bom yes)
+		(on_board yes)
+		(dnp no)
+		(property "Reference" "U5"
+			(at 55 91 0)
+			(effects (font (size 1.27 1.27)))
+		)
+		(property "Value" "DW01A"
+			(at 55 93 0)
+			(effects (font (size 1.27 1.27)))
+		)
+		(property "Footprint" "Package_TO_SOT_SMD:SOT-23-6"
+			(at 55 100 0)
+			(effects (font (size 1.27 1.27)) (hide yes))
+		)
+		(property "Datasheet" "~"
+			(at 55 100 0)
+			(effects (font (size 1.27 1.27)) (hide yes))
+		)
+		(property "Description" ""
+			(at 55 100 0)
+			(effects (font (size 1.27 1.27)) (hide yes))
+		)
+		(pin "1")
+		(pin "2")
+		(pin "3")
+		(pin "4")
+		(pin "5")
+		(pin "6")
+		(instances
+			(project ""
+				(path "/voice-car-001"
+					(reference "U5")
+					(unit 1)
+				)
+			)
+		)
+	)
+	(symbol
+		(lib_id "Custom:FS8205A")
+		(at 75 100 0)
+		(unit 1)
+		(exclude_from_sim no)
+		(in_bom yes)
+		(on_board yes)
+		(dnp no)
+		(property "Reference" "Q1"
+			(at 75 91 0)
+			(effects (font (size 1.27 1.27)))
+		)
+		(property "Value" "FS8205A"
+			(at 75 93 0)
+			(effects (font (size 1.27 1.27)))
+		)
+		(property "Footprint" "Package_TO_SOT_SMD:SOT-23-6"
+			(at 75 100 0)
+			(effects (font (size 1.27 1.27)) (hide yes))
+		)
+		(property "Datasheet" "~"
+			(at 75 100 0)
+			(effects (font (size 1.27 1.27)) (hide yes))
+		)
+		(property "Description" ""
+			(at 75 100 0)
+			(effects (font (size 1.27 1.27)) (hide yes))
+		)
+		(pin "1")
+		(pin "2")
+		(pin "3")
+		(pin "4")
+		(pin "5")
+		(pin "6")
+		(instances
+			(project ""
+				(path "/voice-car-001"
+					(reference "Q1")
+					(unit 1)
+				)
+			)
+		)
+	)
+	(symbol
+		(lib_id "Device:R")
+		(at 55 120 0)
+		(unit 1)
+		(exclude_from_sim no)
+		(in_bom yes)
+		(on_board yes)
+		(dnp no)
+		(property "Reference" "R6"
+			(at 57.28 120 90)
+			(effects (font (size 1.27 1.27)))
+		)
+		(property "Value" "100k"
+			(at 55 120 90)
+			(effects (font (size 1.27 1.27)))
+		)
+		(property "Footprint" "Resistor_SMD:R_0402_1005Metric"
+			(at 55 120 0)
+			(effects (font (size 1.27 1.27)) (hide yes))
+		)
+		(property "Datasheet" "~"
+			(at 55 120 0)
+			(effects (font (size 1.27 1.27)) (hide yes))
+		)
+		(property "Description" "VBAT ADC divider high (VBAT → ADC)"
+			(at 55 120 0)
+			(effects (font (size 1.27 1.27)) (hide yes))
+		)
+		(pin "1")
+		(pin "2")
+		(instances
+			(project ""
+				(path "/voice-car-001"
+					(reference "R6")
+					(unit 1)
+				)
+			)
+		)
+	)
+	(symbol
+		(lib_id "Device:R")
+		(at 55 127 0)
+		(unit 1)
+		(exclude_from_sim no)
+		(in_bom yes)
+		(on_board yes)
+		(dnp no)
+		(property "Reference" "R7"
+			(at 57.28 127 90)
+			(effects (font (size 1.27 1.27)))
+		)
+		(property "Value" "47k"
+			(at 55 127 90)
+			(effects (font (size 1.27 1.27)))
+		)
+		(property "Footprint" "Resistor_SMD:R_0402_1005Metric"
+			(at 55 127 0)
+			(effects (font (size 1.27 1.27)) (hide yes))
+		)
+		(property "Datasheet" "~"
+			(at 55 127 0)
+			(effects (font (size 1.27 1.27)) (hide yes))
+		)
+		(property "Description" "VBAT ADC divider low (ADC → GND)"
+			(at 55 127 0)
+			(effects (font (size 1.27 1.27)) (hide yes))
+		)
+		(pin "1")
+		(pin "2")
+		(instances
+			(project ""
+				(path "/voice-car-001"
+					(reference "R7")
+					(unit 1)
+				)
+			)
+		)
+	)
+	(label "BATT_RAW"
+		(at 62.5 99.76 0)
+		(effects (font (size 1.27 1.27)) (justify left bottom))
+	)
+	(label "BATT_RAW"
+		(at 68.0 97.5 0)
+		(effects (font (size 1.27 1.27)) (justify left bottom))
+	)
+	(label "VBAT_MON"
+		(at 55.0 122.0 0)
+		(effects (font (size 1.27 1.27)) (justify left bottom))
+	)
+	(label "VBAT_MON"
+		(at 140.0 27.46 0)
+		(effects (font (size 1.27 1.27)) (justify left bottom))
+	)
+	(text "Battery protection: DW01A + FS8205A\nBATT_RAW: unprotected battery input\nVBAT: protected output to rest of circuit\nVBAT_MON → ESP32 GPIO10 (ADC1_CH9)\nVBAT_MON = VBAT × 47/(100+47) ≈ VBAT × 0.32\nLow battery threshold: VBAT_MON < 1.06V → VBAT < 3.3V"
+		(at 55 135 0)
+		(effects (font (size 1.27 1.27)) (justify left))
+	)
 )
