File: electronics/rove_sv/rove_sv.kicad_sch (KiCad schematic)
At the start: 0 parts

Commit message: Add ROVE-SV schematic and PCB (servo + voice variant)
Derived from ROVE-V using tools/create_rove_sv.py:
- ESP32-S3 IO8 (y=112.54) → SERVO1 PWM signal
- ESP32-S3 IO9 (y=115.08) → SERVO2 PWM signal
- J5/J6 added: 3-pin PinHeader_1x03_P2.54mm (GND/VBAT/SIG)
- PCB footprints placed at (50,42) and (50,47); routing TBD

All ROVE-V circuits preserved: DRV8833 motors, INMP441 mic,
DW01A+FS8205A battery protection, XC6220 LDO, USB-C

Co-Authored-By: Claude Sonnet 4.6 <noreply@anthropic.com>
Parts:
- added C1, C3: 10uF, Capacitor_SMD:CP_Elec_6.3x5.8, symbol Device:C_Polarized_Small
- added C2, C4, C7, C8: 0.1uF, Capacitor_SMD:C_0805_2012Metric, symbol Device:C_Small
- added C5: 100uF, Capacitor_SMD:CP_Elec_6.3x5.8, symbol Device:C_Polarized_Small
- added C6: 10nF, Capacitor_SMD:C_0805_2012Metric, symbol Device:C_Small
- added D1: Blue, LED_SMD:LED_0805_2012Metric, symbol Device:LED
- added D2, D3: SS14, Diode_SMD:D_SOD-123, symbol Device:D_Schottky
- added J1: USB-C, Connector_USB:USB_C_Receptacle_HRO_TYPE-C-31-M-12, symbol Connector:USB_C_Receptacle_USB2.0_16P
- added J2: Battery, Connector_JST:JST_PH_B2B-PH-K_1x02_P2.00mm_Vertical, symbol Connector_Generic:Conn_01x02
- added J3: LeftMotor, Connector_JST:JST_PH_B2B-PH-K_1x02_P2.00mm_Vertical, symbol Connector_Generic:Conn_01x02
- added J4: RightMotor, Connector_JST:JST_PH_B2B-PH-K_1x02_P2.00mm_Vertical, symbol Connector_Generic:Conn_01x02
- added J5: Servo1, Connector_PinHeader_2.54mm:PinHeader_1x03_P2.54mm_Vertical, symbol Connector_Generic:Conn_01x03
- added J6: Servo2, Connector_PinHeader_2.54mm:PinHeader_1x03_P2.54mm_Vertical, symbol Connector_Generic:Conn_01x03
- added MK1: INMP441, Microphone:Knowles_LGA-6_3.76x4.72mm, symbol Custom:INMP441
- added Q1: FS8205A, Package_TO_SOT_SMD:SOT-23-6, symbol Custom:FS8205A
- added R1, R2, R6: 10k, Resistor_SMD:R_0805_2012Metric, symbol Device:R
- added R3: 330, Resistor_SMD:R_0805_2012Metric, symbol Device:R
- added R4, R5: 5.1k, Resistor_SMD:R_0805_2012Metric, symbol Device:R
- added R6: 100k, Resistor_SMD:R_0402_1005Metric, symbol Device:R
- added R7: 47k, Resistor_SMD:R_0402_1005Metric, symbol Device:R
- added SW1: BOOT, Button_Switch_SMD:SW_SPST_SKQG_WithoutStem, symbol Switch:SW_Push
- added SW2: RST, Button_Switch_SMD:SW_SPST_SKQG_WithoutStem, symbol Switch:SW_Push
- added U1: ESP32-S3-WROOM-1, RF_Module:ESP32-S3-WROOM-1, symbol RF_Module:ESP32-S3-WROOM-1
- added U2: XC6220B331MR, Package_TO_SOT_SMD:SOT-23-5, symbol Regulator_Linear:XC6220B331MR
- added U3: DRV8833PW, Package_SO:TSSOP-16_4.4x5mm_P0.65mm, symbol Driver_Motor:DRV8833PW
- added U5: DW01A, Package_TO_SOT_SMD:SOT-23-6, symbol Custom:DW01A
Connections:
- new net: J1.A4 (VBUS), J1.A9 (VBUS), J1.B4 (VBUS), J1.B9 (VBUS)
- new net 3V3: C2.1, C3.1, C4.1, R1.1, R2.1, R6.1, U1.2 (3V3), U2.5 (VOUT)
- new net AOUT1: J3.1 (Pin_1), U3.2 (AOUT1)
- new net AOUT2: J3.2 (Pin_2), U3.4 (AOUT2)
- new net BOUT1: J4.1 (Pin_1), U3.7 (BOUT1)
- new net BOUT2: J4.2 (Pin_2), U3.5 (BOUT2)
- new net CC1: J1.A5 (CC1), R4.1
- new net CC2: J1.B5 (CC2), R5.1
- new net DRV_SLEEP: R6.2, U3.1 (~{SLEEP})
- new net EN: R1.2, SW2.1, U1.3 (EN)
- new net GND: C1.2, C2.2, C3.2, C4.2, C5.2, C7.2, C8.2, D1.1 (K), J1.A1 (GND), J1.A12 (GND), J1.B1 (GND), J1.B12 (GND), J1.S1 (SHIELD), J2.2 (Pin_2), R4.2, R5.2, SW1.2, SW2.2, U1.1 (GND), U1.40 (GND), U1.41 (GND), U2.2 (GND), U3.13 (GND), U3.3 (AISEN), U3.6 (BISEN)
- new net I2S_SCK: U1.33 (IO40)
- new net I2S_SD: MK1.6 (L/R), U1.34 (IO41)
- new net I2S_WS: MK1.1 (VDD), U1.32 (IO39)
- new net IO0: R2.2, SW1.1, U1.27 (IO0)
- new net LED_ANODE: D1.2 (A), R3.2
- new net LEFT_IN1: U1.4 (IO4), U3.16 (AIN1)
- new net LEFT_IN2: U1.5 (IO5), U3.15 (AIN2)
- new net RIGHT_IN1: U1.6 (IO6), U3.9 (BIN1)
- new net RIGHT_IN2: U1.7 (IO7), U3.10 (BIN2)
- new net SERVO1: U1.12 (IO8)
- new net SERVO2: U1.17 (IO9)
- new net STATUS_LED: R3.1, U1.18 (IO10)
- new net USB_5V: D2.2 (A)
- new net USB_D+: J1.A6 (D+), J1.B6 (D+), U1.14 (USB_D+)
- new net USB_D-: J1.A7 (D-), J1.B7 (D-), U1.13 (USB_D-)
- new net VBAT_MOTOR: C5.1, C6.1, C6.2, C8.1, D3.2 (A), J2.1 (Pin_1), U3.11 (VCP), U3.12 (VM)
- new net VINT: C7.1, U3.14 (VINT)
- new net VIN_3V3: C1.1, D2.1 (K), D3.1 (K), U2.1 (VIN), U2.3 (CE)
- no-connect marks 0 -> 62
Other:
- note added: "Battery protection: DW01A + FS8205A BATT_RAW: unprotected battery input VBAT: protected output to rest of circuit VBAT_MON → ESP32 GPIO10 (ADC1_CH9) VBAT_MON = VBAT × 47/(100+47) ≈ VBAT × 0.32 Low battery threshold: VBAT_MON < 1.06V → VBAT < 3.3V"
- note added: "NOTE: TP4056 and INMP441 connections - see docs/schematic_notes.md"
- note added: "['at', '50', '142', '0']"
- note removed: "['at', '50', '50', '0']"
- note removed: "['at', '50', '58', '0']"
- note removed: "['at', '50', '64', '0']"
